File: Presentation/boards/pedalboard-led-ring.kicad_pcb (KiCad board)
At the start: 2 copper layers, 36 x 28 mm, 16 parts, among them J1 Conn_02x03, U1 TLC5973, U2 LT3494AEDDBPBF

Commit message: Deploying to main from @ pedalboard/pedalboard-led-ring@1700bd16053fd4b3e2c698d5dc94816918e5af73 🚀
Parts:
- C2: value 100nF -> 330nF
- C4: value 0.22uF_0603_25V -> 330nF
- moved J1 0.90 mm to (96.5, 68.0)
- moved L1 0.61 mm to (87.9, 67.1)
- moved C3 0.40 mm to (90.0, 71.1)
- moved C4 0.10 mm to (82.9, 69.3)
Connections:
- J1 pad 3: Net-(J1-VLED) -> GND
- J1 pad 4: GND -> Net-(J1-VLED)
- J1 pad 5: Net-(U1-SDI) -> VCC
- J1 pad 6: VCC -> Net-(U1-SDI)
Routing:
- net VCC: track 3.34 -> 5.36 mm
- net GND: track 2.85 -> 1.05 mm, vias 0 -> 10
- net Net-(U1-SDI): track 17.8 -> 16.2 mm
- net Net-(J1-SDO): track 16.1 -> 17.2 mm
- added copper zone on F.Cu, net GND
