File: Presentation/boards/pedalboard-led-ring.kicad_pcb (KiCad board)
At the start: 2 copper layers, 28 x 28 mm, 25 parts, among them J1 Conn_02x02_Odd_Even

Commit message: Deploying to main from @ pedalboard/pedalboard-led-ring@b0111f044335ce82a2366fa9673f79a32cee981a 🚀
Parts:
- added J2: edge, Connector_PinSocket_2.00mm:PinSocket_2x02_P2.00mm_Vertical_SMD, B.Cu at (90.0, 70.0)
- added R1: 330, Resistor_SMD:R_0201_0603Metric_Pad0.64x0.40mm_HandSolder, F.Cu at (88.9, 61.7)
- J1: value Conn_02x02_Odd_Even -> middle
- moved J1 1.00 mm to (90.0, 60.0)
Connections:
- J1 pad 3: Net-(D1-DIN) -> Net-(J1-Pin_3)
Routing:
- net Net-(J1-Pin_3): track 0.00 -> 19.4 mm, vias 0 -> 1
- net Net-(D12-DOUT): track 2.86 -> 12.0 mm
- net GND: track 12.1 -> 7.71 mm
- net Net-(D1-DIN): track 5.17 -> 1.28 mm, vias 1 -> 0
- net VCC: track 19.3 -> 21.0 mm
Other:
- board size 28 x 28 mm -> 30 x 30 mm
