File: Presentation/boards/pedalboard-led-ring.kicad_pcb (KiCad board)
At the start: 2 copper layers, 30 x 30 mm, 27 parts, among them J1 middle, J2 edge

Commit message: Deploying to main from @ pedalboard/pedalboard-led-ring@67a3d3a1d164a125443a7aef7d29769f316d677e 🚀
Parts:
- added H1: MountingHole, MountingHole:MountingHole_2.2mm_M2, F.Cu at (68.0, 72.0)
- added H2: MountingHole, MountingHole:MountingHole_2.2mm_M2, F.Cu at (92.0, 48.0)
- added H3: MountingHole, MountingHole:MountingHole_2.2mm_M2, F.Cu at (68.0, 48.0)
Other:
- board text added: "D0"
- board text added: "DI"
- board text added: "DO"
- board text added: "GND"
- board text added: "VCC"
